File: P0004-PCB-001.kicad_sch (KiCad schematic)
At the start: 19 parts, among them CN1 Liansheng PH--00603, SW1 Khon TSB06331-090D332DA-R0500, SW2 Khon TSB06331-090D332DA-R0500, SW3 Khon TSB06331-090D332DA-R0500, SW4 Khon TSB06331-090D332DA-R0500

Commit message: most things connected
Other:
- sheet Microcontroller ports: added DFU_EN; removed none
Changed lines of the file:
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@@
+			)
+		)
+		(pin "DFU_EN" input
+			(at 99.06 157.48 0)
+			(effects
+				(font
+					(size 1.27 1.27)
+				)
+				(justify right)
 			)
 		)
