File: P0004-PCB-001.kicad_sch (KiCad schematic)
At the start: 19 parts, among them CN1 Liansheng PH--00603, SW1 Khon TSB06331-090D332DA-R0500, SW2 Khon TSB06331-090D332DA-R0500, SW3 Khon TSB06331-090D332DA-R0500, SW4 Khon TSB06331-090D332DA-R0500

Commit message: just need last tidy up
Parts:
- removed H10, H3, H6, H7: Khon SC109AM1, Switch_WUT:Khon_SC109, symbol Switch_WUT:Khon_SC109AM1
- removed SW1, SW2, SW3, SW4: Khon TSB06331-090D332DA-R0500, Switch_WUT:Khon_TSB06331-090, symbol Switch_WUT:Khon_TSB06331-090D332DA-R0500
Connections:
- net VIN: now reaches CN1.1 (Pin_1)
- net 0V: now reaches CN1.10
- net 0V: now also CN1.12, CN1.14, CN1.16, CN1.18, CN1.2 (Pin_1), CN1.20, CN1.22, CN1.24, CN1.26, CN1.28, CN1.3, CN1.30, CN1.4, CN1.6, CN1.8
- net ETH_TX_N: now reaches CN1.11
- net ~{ETH_LINK_OD}: now reaches CN1.13
- net ~{ETH_ACT_OD}: now reaches CN1.15
- net INT_SDA: now reaches CN1.17
- net INT_SCL: now reaches CN1.19
- net USB_P: now reaches CN1.21
- net USB_N: now reaches CN1.23
- net DFU_EN: now reaches CN1.25
- net ~{INT_ALERT}: now reaches CN1.27
- net 3V3_EXPANSION: now reaches CN1.29
- net ETH_RX_P: now reaches CN1.5
- net ETH_RX_N: now reaches CN1.7
- net ETH_TX_P: now reaches CN1.9
Other:
- sheet Microcontroller ports: added USB_DEVICE_N, USB_DEVICE_P, ~{3V3_EXPANSION_FAULT}, ~{INT_ALERT}; removed none
- sheet Power Supplies ports: added ~{3V3_EXPANSION_FAULT}, ~{5V_VBUS_FAULT}; removed ~{VBUS_FAULT}
- moved on the sheet: CN1

Commit message: component tidy up
Parts:
- removed LS1: HNDZ MLT8530, Audio_WUT:HNDZ_MLT8530, symbol Audio_WUT:HNDZ_MLT8530
Changed lines of the file:
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@@
-	)
-	(symbol
-		(lib_id "Audio_WUT:HNDZ_MLT8530")
-		(at 266.7 147.32 0)
-		(unit 1)
-		(body_style 1)
-		(exclude_from_sim no)
-		(in_bom yes)
-		(on_board yes)
-		(in_pos_files yes)
-		(dnp no)
-		(fields_autoplaced yes)
-		(property "Reference" "LS1"
-			(at 271.78 147.3199 0)
-			(show_name no)
-			(do_not_autoplace no)
-			(effects
-				(font
-					(size 1.27 1.27)
-				)
-				(justify left)
-			)
-		)
-		(property "Value" "HNDZ MLT8530"
-			(at 271.78 149.8599 0)
-			(show_name no)
-			(do_not_autoplace no)
-			(effects
-				(font
-					(size 1.27 1.27)
-				)
-				(justify left)
-			)
-		)
-		(property "Footprint" "Audio_WUT:HNDZ_MLT8530"
-			(at 266.7 147.32 0)
-			(hide yes)
-			(show_name no)
-			(do_not_autoplace no)
-			(effects
-				(font
-					(size 1.27 1.27)
-				)
-			)
-		)
-		(property "Datasheet" "https://jlc-prod-smt.oss-eu-central-1.aliyuncs.com/smtDataManualFile/8588881949994074112-C94599.pdf?response-content-disposition=attachment%3B%20filename%3DC94599.pdf%3B%20filename%2A%3DUTF-8%27%27C94599.pdf&x-oss-date=20260606T154850Z&x-oss-expires=1800&x-oss-security-token=CAISgAN1q6Ft5B2yfSjIr5n5IYju1Y9kxfunQ2f0skYvO%2B4VtZecgzz2IHhMdHJsAOodtv0%2FmmhT6PkclqRLcbhpcmfjV%2BZHzLB8qeAS7w1A4J7b16cNrbH4M4H6aXeirtuwDsz9SNTCALjPD3nPii50x5bjaDymRCbLGJaViJlhHLN1Ow6jdmhpCctxLAlvo9NgFxm3D%2Fu2NQPwiWf9FVdhvhEG6Vly8qOi2MaRmFy8yFTx0b0SvJ%2BjYMrmPctoN9JnSdC5mfdzau3a1TJ84gRD0a5wkaVA1zbDs5bfISEIuUzebreLqY03dV4mOvdqIcMe8qigz88fk%2FfIioH6xyxKOexoSCnFTOiiupCcQLPyao9jLu6iayqViY7QaIOTqQohZmkAMwVOasAsI3Ngh4zF97Qt0cVNkXO9gWfLI8DtuMleWhpDH8tN3tHD0eS19jklBdzSlusJRAJJUVBflCeKEaRNSAd3WGhEfM2%2BBt4QT30w5N2u00S8OSMIAGjL%2B6KWD5sagAFEQDONgaycLHLYJ9OE8%2FZjaXFts1t7emH6oRWEhY3rWteXUHjj41EzNWre8odwgMo6BFDtkADd7AiAper%2FazIkwQsNO6ZmdB46Bu32hqnpPFkN4PLaDvlVS1boV0Zqtfrcn1HjoIpuWa%2FGSxylcwHt%2BYbYxQSACHIHM%2BiBFC2JDyAA&x-oss-signature-version=OSS4-HMAC-SHA256&x-oss-credential=STS.NZLj2Z8PEr9LAAEVFz7a9ZR7a%2F20260606%2Feu-central-1%2Foss%2Faliyun_v4_request&x-oss-signature=2cdda2966896dba1043c2287a453b14279a90852679b376f1c24650ecda25bf7"
-			(at 266.7 147.32 0)
-			(hide yes)
-			(show_name no)
-			(do_not_autoplace no)
-			(effects
-				(font
-					(size 1.27 1.27)
-				)
-			)
-		)
-		(property "Description" "Speaker, 8.5x8.5mm, 2.7kHz"
-			(at 266.7 147.32 0)
-			(hide yes)
-			(show_name no)
-			(do_not_autoplace no)
-			(effects
-				(font
-					(size 1.27 1.27)
-				)
-			)
-		)
-		(property "Manufacturer" "Jiangsu Huaneng Elec"
-			(at 266.7 147.32 0)
-			(hide yes)
-			(show_name no)
-			(do_not_autoplace no)
-			(effects
-				(font
-					(size 1.27 1.27)
-				)
-			)
-		)
-		(property "MPN" "MLT-8530"
-			(at 266.7 147.32 0)
-			(hide yes)
-			(show_name no)
-			(do_not_autoplace no)
-			(effects
-				(font
-					(size 1.27 1.27)
-				)
-			)
-		)
-		(property "JLC Order Code" "C94599"
-			(at 266.7 147.32 0)
-			(hide yes)
-			(show_name no)
-			(do_not_autoplace no)
-			(effects
-				(font
-					(size 1.27 1.27)
-				)
-			)
-		)
-		(pin "2"
-		)
-		(pin "1"
-		)
-		(pin "3"
-		)
-		(pin "4"
-		)
-		(instances
-			(project "P0004-PCB-001"
-				(path "/acdb93e6-9aa6-4a78-8a68-9d0ae3318f45"
-					(reference "LS1")
-					(unit 1)
-				)
-			)
-		)
 	)
 	(symbol

Commit message: added tidied up library symbols
Parts:
- renumbered H4 to H3, H5 to H4, H8 to H5, H9 to H6, H11 to H7, H12 to H8, H13 to H9
Changed lines of the file:
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@@
 		(dnp no)
 		(fields_autoplaced yes)
-		(property "Reference" "#PWR0114"
+		(property "Reference" "#PWR02"
 			(at 185.42 142.24 0)
 			(hide yes)
@@
 			(project "P0004-PCB-001"
 				(path "/acdb93e6-9aa6-4a78-8a68-9d0ae3318f45"
-					(reference "#PWR0114")
+					(reference "#PWR02")
 					(unit 1)
 				)
@@
 		(dnp no)
 		(fields_autoplaced yes)
-		(property "Reference" "H9"
+		(property "Reference" "H6"
 			(at 96.52 125.73 0)
 			(show_name no)
@@
 			(project "P0004-PCB-001"
 				(path "/acdb93e6-9aa6-4a78-8a68-9d0ae3318f45"
-					(reference "H9")
+					(reference "H6")
 					(unit 1)
 				)
@@
 		(dnp no)
 		(fields_autoplaced yes)
-		(property "Reference" "H5"
+		(property "Reference" "H4"
 			(at 77.47 125.73 0)
 			(show_name no)
@@
 			(project "P0004-PCB-001"
 				(path "/acdb93e6-9aa6-4a78-8a68-9d0ae3318f45"
-					(reference "H5")
+					(reference "H4")
 					(unit 1)
 				)
@@
 		(dnp no)
 		(fields_autoplaced yes)
-		(property "Reference" "H11"
+		(property "Reference" "H7"
 			(at 114.3 115.57 0)
 			(show_name no)
@@
 			(project "P0004-PCB-001"
 				(path "/acdb93e6-9aa6-4a78-8a68-9d0ae3318f45"
-					(reference "H11")
+					(reference "H7")
 					(unit 1)
 				)
@@
 		(dnp no)
 		(fields_autoplaced yes)
-		(property "Reference" "H8"
+		(property "Reference" "H5"
 			(at 96.52 115.57 0)
 			(show_name no)
@@
 			(project "P0004-PCB-001"
 				(path "/acdb93e6-9aa6-4a78-8a68-9d0ae3318f45"
-					(reference "H8")
+					(reference "H5")
 					(unit 1)
 				)
@@
 		(dnp no)
 		(fields_autoplaced yes)
-		(property "Reference" "H4"
+		(property "Reference" "H3"
 			(at 77.47 115.57 0)
 			(show_name no)
@@
 			(project "P0004-PCB-001"
 				(path "/acdb93e6-9aa6-4a78-8a68-9d0ae3318f45"
-					(reference "H4")
+					(reference "H3")
 					(unit 1)
 				)
@@
 		(dnp no)
 		(fields_autoplaced yes)
-		(property "Reference" "#PWR0115"
+		(property "Reference" "#PWR01"
 			(at 169.545 147.955 0)
 			(hide yes)
@@
 			(project "P0004-PCB-001"
 				(path "/acdb93e6-9aa6-4a78-8a68-9d0ae3318f45"
-					(reference "#PWR0115")
+					(reference "#PWR01")
 					(unit 1)
 				)
@@
 		(dnp no)
 		(fields_autoplaced yes)
-		(property "Reference" "H13"
+		(property "Reference" "H9"
 			(at 281.94 270.5099 0)
 			(show_name no)
@@
 			(project "P0004-PCB-001"
 				(path "/acdb93e6-9aa6-4a78-8a68-9d0ae3318f45"
-					(reference "H13")
+					(reference "H9")
 					(unit 1)
 				)
@@
 		(dnp no)
 		(fields_autoplaced yes)
-		(property "Reference" "H12"
+		(property "Reference" "H8"
 			(at 114.3 125.73 0)
 			(show_name no)
@@
 			(project "P0004-PCB-001"
 				(path "/acdb93e6-9aa6-4a78-8a68-9d0ae3318f45"
-					(reference "H12")
+					(reference "H8")
 					(unit 1)
 				)
@@
 		(dnp no)
 		(fields_autoplaced yes)
-		(property "Reference" "#PWR0113"
+		(property "Reference" "#PWR03"
 			(at 205.74 142.24 0)
 			(hide yes)
@@
 			(project "P0004-PCB-001"
 				(path "/acdb93e6-9aa6-4a78-8a68-9d0ae3318f45"
-					(reference "#PWR0113")
+					(reference "#PWR03")
 					(unit 1)
 				)

Commit message: draft v1 release
Other:
- sheet Microcontroller ports: added INT_SCL, INT_SDA; removed none
