File: power.kicad_sch (KiCad schematic)
At the start: 37 parts, among them U5 TI LMR54410DBV, U6 TI LMR54410DBV, U7 TI TPS2553DBV

Commit message: just need last tidy up
Parts:
- removed R21: 47k, Resistor_WUT:R_0402_1005Metric, symbol resistor_auto_wut:KOA Speer RK73H1ETTP4702F
- removed R32, R33, R34, R4: 1k0, Resistor_WUT:R_0402_1005Metric, symbol aaa_resistor_auto_wut:KOA Speer RK73H1ETTP1001F
- added C49: 100n, Capacitor_WUT:C_0402_1005Metric, symbol aaa_capacitor_auto_wut:Yageo CC0402KRX7R8BB104
- added C50: 22u, Capacitor_SMD:C_0603_1608Metric, symbol aaa_capacitor_auto_wut:Murata GRM188R61C226ME01
- added R21: 82k, Resistor_WUT:R_0402_1005Metric, symbol resistor_auto_wut:KOA Speer RK73H1ETTP8202F
- added R59: 47k, Resistor_WUT:R_0402_1005Metric, symbol resistor_auto_wut:KOA Speer RK73H1ETTP4702F
- added R60: 10k, Resistor_WUT:R_0402_1005Metric, symbol aaa_resistor_auto_wut:KOA Speer RK73H1ETTP1002F
- added U8: TI TPS2553DBVR-1, IC_WUT:SOT-23-6, symbol IC_WUT:TPS2553DBVR-1
- C43, C44: value 15p -> 18p; symbol capacitor_auto_wut:Kemet C0402C150G5GACTU -> capacitor_auto_wut:Kemet C0402C180K3GACTU; MPN C0402C150G5GACTU -> C0402C180K3GACTU; Tolerance 2% -> 10%; Voltage 50V -> 25V
- U7: value TI TPS2553DBV -> TI TPS2553DBVR-1; symbol IC_WUT:TPS2553DBV -> IC_WUT:TPS2553DBVR-1; MPN TPS2553DBV -> TPS2553DBVR-1
Connections:
- net 0V: now also C49.2, C50.2, R59.2, U8.2 (GND)
- net 3V3: now also C49.1, R60.1, U8.1 (IN), U8.3 (EN)
- net VOUT_5V: now also R21.1
- net at C44.2, R22.1, U6.3 (FB): now also R21.2
- net ~{VBUS_FAULT} renamed ~{5V_VBUS_FAULT}
- new net: R59.1, U8.5 (ILIM)
- new net 3V3_EXPANSION: C50.1, U8.6 (OUT)
- new net ~{3V3_EXPANSION_FAULT}: R60.2, U8.4 (~{FAULT})
Other:
- note added: "3V3 Expansion Load Switch"
- note added: "Vfb = 0.8V Vout = 0.8 * (1+82/15) = 5.17V"
- note removed: "TODO Feedback resistors"
- note removed: "TODO Replace with 0402 LEDs"
