File: power.kicad_sch (KiCad schematic)
At the start: 38 parts, among them U5 TI LMR54410DBV, U6 TI LMR54410DBV, U7 TI TPS2553DBVR-1, U8 TI TPS2553DBVR-1

Commit message: component tidy up
Parts:
- removed D11: 15V, Diode_SMD:D_SOD-323, symbol tvs_zener_auto_wut:Bourns CDSOD323-T15S
- added D15: 15V, Diode_WUT:D_SOD-323, symbol tvs_zener_auto_wut:Bourns CDSOD-323-T15S
- C35, C36, C39, C40, C41, C42, C50: footprint Capacitor_SMD:C_0603_1608Metric -> Capacitor_WUT:C_0603_1608Metric
- D12, D13: footprint Diode_SMD:D_SOD-523 -> Diode_WUT:D_SOD-523
- F2, F3, F4: footprint Fuse:Fuse_0603_1608Metric -> Fuse_WUT:Fuse_0603_1608Metric
Connections:
- net 0V: now also D15.2 (A)
- net VIN_SAFE: now also D15.1 (K)
Changed lines of the file:
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@@
 			)
 		)
-		(property "Footprint" "Capacitor_SMD:C_0603_1608Metric"
+		(property "Footprint" "Capacitor_WUT:C_0603_1608Metric"
 			(at 167.64 172.72 0)
 			(hide yes)
@@
 			)
 		)
-		(property "Footprint" "Capacitor_SMD:C_0603_1608Metric"
+		(property "Footprint" "Capacitor_WUT:C_0603_1608Metric"
 			(at 154.94 172.72 0)
 			(hide yes)
@@
 			)
 		)
-		(property "Footprint" "Capacitor_SMD:C_0603_1608Metric"
+		(property "Footprint" "Capacitor_WUT:C_0603_1608Metric"
 			(at 142.24 172.72 0)
 			(hide yes)
@@
 	)
 	(symbol
+		(lib_id "tvs_zener_auto_wut:Bourns CDSOD-323-T15S")
+		(at 45.72 60.96 90)
+		(unit 1)
+		(body_style 1)
+		(exclude_from_sim no)
+		(in_bom yes)
+		(on_board yes)
+		(in_pos_files yes)
+		(dnp no)
+		(fields_autoplaced yes)
+		(property "Reference" "D15"
+			(at 48.26 59.4359 90)
+			(show_name no)
+			(do_not_autoplace no)
+			(effects
+				(font
+					(size 1.27 1.27)
+				)
+				(justify right)
+			)
+		)
+		(property "Value" "15V"
+			(at 48.26 61.9759 90)
+			(show_name no)
+			(do_not_autoplace no)
+			(effects
+				(font
+					(size 1.27 1.27)
+				)
+				(justify right)
+			)
+		)
+		(property "Footprint" "Diode_WUT:D_SOD-323"
+			(at 45.72 60.96 0)
+			(hide yes)
+			(show_name no)
+			(do_not_autoplace no)
+			(effects
+				(font
+					(size 1.27 1.27)
+				)
+			)
+		)
+		(property "Datasheet" "https://www.mouser.co.uk/datasheet/2/54/cdSOD-323_txxsc-777083.pdf"
+			(at 45.72 60.96 0)
+			(hide yes)
+			(show_name no)
+			(do_not_autoplace no)
+			(effects
+				(font
+					(size 1.27 1.27)
+				)
+			)
+		)
+		(property "Description" "15V SOD-323 TVS Diode"
+			(at 45.72 60.96 0)
+			(hide yes)
+			(show_name no)
+			(do_not_autoplace no)
+			(effects
+				(font
+					(size 1.27 1.27)
+				)
+			)
+		)
+		(property "Manufacturer" "Bourns"
+			(at 45.72 60.96 0)
+			(hide yes)
+			(show_name no)
+			(do_not_autoplace no)
+			(effects
+				(font
+					(size 1.27 1.27)
+				)
+			)
+		)
+		(property "MPN" "CDSOD-323-T15S"
+			(at 45.72 60.96 0)
+			(hide yes)
+			(show_name no)
+			(do_not_autoplace no)
+			(effects
+				(font
+					(size 1.27 1.27)
+				)
+			)
+		)
+		(property "Height" "1.14mm"
+			(at 45.72 60.96 0)
+			(hide yes)
+			(show_name no)
+			(do_not_autoplace no)
+			(effects
+				(font
+					(size 1.27 1.27)
+				)
+			)
+		)
+		(pin "1"
+		)
+		(pin "2"
+		)
+		(instances
+			(project "P0004-PCB-001"
+				(path "/acdb93e6-9aa6-4a78-8a68-9d0ae3318f45/35d58bcc-6ce4-4583-93f1-63aee4dbfc17"
+					(reference "D15")
+					(unit 1)
+				)
+			)
+		)
+	)
+	(symbol
 		(lib_id "Power_WUT:0V")
 		(at 289.56 180.34 0)
@@
 			)
 		)
-		(property "Footprint" "Diode_SMD:D_SOD-523"
+		(property "Footprint" "Diode_WUT:D_SOD-523"
 			(at 213.36 66.04 0)
 			(hide yes)
@@
 			)
 		)
-		(property "Description" "5V SOD523 TVS Diode"
+		(property "Description" "5V SOD-523 TVS Diode"
 			(at 213.36 66.04 0)
 			(hide yes)
@@
 			)
 		)
-		(property "Footprint" "Capacitor_SMD:C_0603_1608Metric"
+		(property "Footprint" "Capacitor_WUT:C_0603_1608Metric"
 			(at 180.34 172.72 0)
 			(hide yes)
@@
 			)
 		)
-		(property "Footprint" "Fuse:Fuse_0603_1608Metric"
+		(property "Footprint" "Fuse_WUT:Fuse_0603_1608Metric"
 			(at 38.1 53.34 0)
 			(hide yes)
@@
 			)
 		)
-		(property "Footprint" "Capacitor_SMD:C_0603_1608Metric"
+		(property "Footprint" "Capacitor_WUT:C_0603_1608Metric"
 			(at 172.72 66.04 0)
 			(hide yes)
@@
 	)
 	(symbol
-		(lib_id "tvs_zener_auto_wut:Bourns CDSOD323-T15S")
-		(at 45.72 60.96 90)
-		(unit 1)
-		(body_style 1)
-		(exclude_from_sim no)
-		(in_bom yes)
-		(on_board yes)
-		(in_pos_files yes)
-		(dnp no)
-		(fields_autoplaced yes)
-		(property "Reference" "D11"
-			(at 48.26 59.4359 90)
-			(show_name no)
-			(do_not_autoplace no)
-			(effects
-				(font
-					(size 1.27 1.27)
-				)
-				(justify right)
-			)
-		)
-		(property "Value" "15V"
-			(at 48.26 61.9759 90)
-			(show_name no)
-			(do_not_autoplace no)
-			(effects
-				(font
-					(size 1.27 1.27)
-				)
-				(justify right)
-			)
-		)
-		(property "Footprint" "Diode_SMD:D_SOD-323"
-			(at 45.72 60.96 0)
-			(hide yes)
-			(show_name no)
-			(do_not_autoplace no)
-			(effects
-				(font
-					(size 1.27 1.27)
-				)
-			)
-		)
-		(property "Datasheet" "https://www.mouser.co.uk/datasheet/2/54/cdsod323_txxsc-777083.pdf"
-			(at 45.72 60.96 0)
-			(hide yes)
-			(show_name no)
-			(do_not_autoplace no)
-			(effects
-				(font
-					(size 1.27 1.27)
-				)
-			)
-		)
-		(property "Description" "15V SOD323 TVS Diode"
-			(at 45.72 60.96 0)
-			(hide yes)
-			(show_name no)
-			(do_not_autoplace no)
-			(effects
-				(font
-					(size 1.27 1.27)
-				)
-			)
-		)
-		(property "Manufacturer" "Bourns"
-			(at 45.72 60.96 0)
-			(hide yes)
-			(show_name no)
-			(do_not_autoplace no)
-			(effects
-				(font
-					(size 1.27 1.27)
-				)
-			)
-		)
-		(property "MPN" "CDSOD323-T15S"
-			(at 45.72 60.96 0)
-			(hide yes)
-			(show_name no)
-			(do_not_autoplace no)
-			(effects
-				(font
-					(size 1.27 1.27)
-				)
-			)
-		)
-		(property "Height" "1.14mm"
-			(at 45.72 60.96 0)
-			(hide yes)
-			(show_name no)
-			(do_not_autoplace no)
-			(effects
-				(font
-					(size 1.27 1.27)
-				)
-			)
-		)
-		(pin "2"
-		)
-		(pin "1"
-		)
-		(instances
-			(project "P0004-PCB-001"
-				(path "/acdb93e6-9aa6-4a78-8a68-9d0ae3318f45/35d58bcc-6ce4-4583-93f1-63aee4dbfc17"
-					(reference "D11")
-					(unit 1)
-				)
-			)
-		)
-	)
-	(symbol
 		(lib_id "inductor_auto_wut:APV ANR4030T100M")
 		(at 147.32 114.3 90)
@@
 			)
 		)
-		(property "Footprint" "Capacitor_SMD:C_0603_1608Metric"
+		(property "Footprint" "Capacitor_WUT:C_0603_1608Metric"
 			(at 289.56 172.72 0)
 			(hide yes)
@@
 			)
 		)
-		(property "Footprint" "Capacitor_SMD:C_0603_1608Metric"
+		(property "Footprint" "Capacitor_WUT:C_0603_1608Metric"
 			(at 172.72 121.92 0)
 			(hide yes)
@@
 			)
 		)
-		(property "Footprint" "Diode_SMD:D_SOD-523"
+		(property "Footprint" "Diode_WUT:D_SOD-523"
 			(at 215.9 121.92 0)
 			(hide yes)
@@
 			)
 		)
-		(property "Description" "5V SOD523 TVS Diode"
+		(property "Description" "5V SOD-523 TVS Diode"
 			(at 215.9 121.92 0)
 			(hide yes)
@@
 			)
 		)
-		(property "Footprint" "Fuse:Fuse_0603_1608Metric"
+		(property "Footprint" "Fuse_WUT:Fuse_0603_1608Metric"
 			(at 208.28 114.3 0)
 			(hide yes)
@@
 			)
 		)
-		(property "Footprint" "Fuse:Fuse_0603_1608Metric"
+		(property "Footprint" "Fuse_WUT:Fuse_0603_1608Metric"
 			(at 205.74 58.42 0)
 			(hide yes)

Commit message: added tidied up library symbols
Parts:
- renumbered C30 to C35, C31 to C36, C32 to C37, C33 to C38, C34 to C39, C35 to C40, C36 to C41, C37 to C42, C38 to C43, C39 to C44, C40 to C45, C41 to C46, C42 to C47, C43 to C48, C44 to C49, C49 to C50, C50 to C51, D15 to D16, D12 to D17, D13 to D18, R16 to R49, R17 to R50, R18 to R51, R19 to R52, R20 to R53, R21 to R54, R22 to R55, R59 to R56, R60 to R57

Commit message: draft v1 release
Other:
- note removed: "TODO input cap"
- moved on the sheet: C35, C36, C37, C38, C39, C40, C41, C42, C43, C44, C45, C46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
