File: microcontroller.kicad_sch (KiCad schematic)
At the start: 85 parts, among them CN10 JST BM06B-SRSS-TB(LF)(SN), CN11 BM05B-SRSS-TB(LF)(SN), CN2 Samtec FTSH-107-01-L-DV-K, CN3 104031-0811, CN4 M20-9990346, CN5 Molex 105057-0001, CN6 BM03B-SRSS-TB(LF)(SN), CN7 BM04B-SRSS-TB(LF)(SN), CN8 BM04B-SRSS-TB(LF)(SN), CN9 JST BM06B-SRSS-TB(LF)(SN), U2 STM32H743VIT6, U3 TMP102AIDRL, U4 Microchip 24AA256UIDT-I/ST

Commit message: just need last tidy up
Parts:
- added D14, D15, D16, D17: 5V, Diode_SMD:D_SOD-523, symbol aaa_tvs_zener_auto_wut:hongjiacheng H5VND5U
- added H10, H3, H6, H7: Khon SC109AM1, Switch_WUT:Khon_SC109, symbol Switch_WUT:Khon_SC109AM1
- added SW1, SW2, SW3, SW4: Khon TSB06331-090D332DA-R0500, Switch_WUT:Khon_TSB06331-090, symbol Switch_WUT:Khon_TSB06331-090D332DA-R0500
- C45: value 10u -> 22u; symbol aaa_capacitor_auto_wut:Samsung Electro-Mechanics CL10A106MO8NQNC -> aaa_capacitor_auto_wut:Murata GRM188R61C226ME01; Height 0.9mm -> 1mm; MPN CL10A106MO8NQNC -> GRM188R61C226ME01; Manufacturer Samsung Electro-Mechanics -> Murata
- D1, D2, D3, D4, D5, D6, D7, D8, D9: value 3V3 -> 5V; symbol aaa_tvs_zener_auto_wut:nexperia PESD3V3U1UB,115 -> aaa_tvs_zener_auto_wut:hongjiacheng H5VND5U; Height 0.65mm -> 0.77mm; MPN PESD3V3U1UB,115 -> H5VND5U; Manufacturer nexperia -> hongjiacheng
Connections:
- net 0V: now also D14.2 (A), D15.2 (A), D16.2 (A), D17.2 (A), SW1.2, SW2.3, SW2.4, SW3.3, SW3.4, SW4.3, SW4.4
- net ~{3V3_EXPANSION_FAULT}: now reaches U2.38 (PE8)
- net ~{SW3}: now reaches U2.39 (PE9)
- net ~{SW3}: now also D16.1 (K), SW3.1
- net ~{SW1}: now reaches U2.40 (PE10)
- net ~{SW1}: now also D14.1 (K), SW1.3
- net ~{SW2}: now reaches U2.42 (PE12)
- net ~{SW2}: now also D15.1 (K), SW2.2
- net ~{SW4}: now reaches U2.43 (PE13)
- net ~{SW4}: now also D17.1 (K), SW4.1
- net USB_DEVICE_D_N renamed USB_DEVICE_N
- net USB_DEVICE_D_P renamed USB_DEVICE_P
- no-connect marks 5 -> 10

Commit message: component tidy up
Parts:
- added C51: 22u, Capacitor_WUT:C_0603_1608Metric, symbol aaa_capacitor_auto_wut:Murata GRM188R61C226ME01
- added D19: B2020WS, Diode_WUT:D_SOD-323, symbol diode_auto_wut:JSCJ B2020WS
- added LS1: Fusheng FUET-5020, Audio_WUT:Fusheng_FUET-5020, symbol Audio_WUT:Fusheng_FUET-5020
- added Q1: BC847C,215, IC_WUT:SOT-23, symbol Transistor_WUT:nexperia_BC847C,215
- added R32: 1k0, Resistor_WUT:R_0402_1005Metric, symbol aaa_resistor_auto_wut:KOA Speer RK73H1ETTP1001F
- C16, C45: footprint Capacitor_SMD:C_0603_1608Metric -> Capacitor_WUT:C_0603_1608Metric
- D1, D14, D15, D16, D17, D2, D3, D4, D5, D6, D7, D8, D9: footprint Diode_SMD:D_SOD-523 -> Diode_WUT:D_SOD-523
- D10: footprint Package_TO_SOT_SMD:SOT-666 -> IC_WUT:SOT-666
- F1: footprint Fuse:Fuse_0603_1608Metric -> Fuse_WUT:Fuse_0603_1608Metric
Connections:
- net 0V: now also C51.2, Q1.2 (E)
- net 3V3: now also C51.1, D19.1 (K), LS1.1 (+)
- net PC5: now reaches U2.33 (PC5)
- net PC5: now also R54.1
- net PB0 renamed SPEAKER
- net SPEAKER: now also R32.1; no longer R54.1
- new net: Q1.1 (B), R32.2
- new net: D19.2 (A), LS1.2 (-), Q1.3 (C)
