File: microcontroller.kicad_sch (KiCad schematic)
At the start: 102 parts, among them CN10 JST BM06B-SRSS-TB(LF)(SN), CN11 BM05B-SRSS-TB(LF)(SN), CN2 Samtec FTSH-107-01-L-DV-K, CN3 104031-0811, CN4 M20-9990346, CN5 Molex 105057-0001, CN6 BM03B-SRSS-TB(LF)(SN), CN7 BM04B-SRSS-TB(LF)(SN), CN8 BM04B-SRSS-TB(LF)(SN), CN9 JST BM06B-SRSS-TB(LF)(SN), Q1 BC847C,215, SW1 Khon TSB06331-090D332DA-R0500, SW2 Khon TSB06331-090D332DA-R0500, SW3 Khon TSB06331-090D332DA-R0500, SW4 Khon TSB06331-090D332DA-R0500, U2 STM32H743VIT6, U3 TMP102AIDRL, U4 Microchip 24AA256UIDT-I/ST

Commit message: added tidied up library symbols
Parts:
- CN10: renamed from CN9; value JST BM06B-SRSS-TB(LF)(SN) -> BM06B-SRSS-TB(LF)(SN); footprint Connector_JST:JST_SH_BM06B-SRSS-TB_1x06-1MP_P1.00mm_Vertical -> Connector_JST_WUT:BM06B-SRSS-TB; symbol Connector_WUT:Header_JST_BM06B-SRSS-TB(LF)(SN) -> connector_auto_wut:JST_BM06B-SRSS-TB(LF)(SN); MPN JST_BM06B-SRSS-TB(LF)(SN) -> BM06B-SRSS-TB(LF)(SN)
- CN11: renamed from CN10; value JST BM06B-SRSS-TB(LF)(SN) -> BM06B-SRSS-TB(LF)(SN); footprint Connector_JST:JST_SH_BM06B-SRSS-TB_1x06-1MP_P1.00mm_Vertical -> Connector_JST_WUT:BM06B-SRSS-TB; symbol Connector_WUT:Header_JST_BM06B-SRSS-TB(LF)(SN) -> connector_auto_wut:JST_BM06B-SRSS-TB(LF)(SN); MPN JST_BM06B-SRSS-TB(LF)(SN) -> BM06B-SRSS-TB(LF)(SN)
- CN3: renamed from CN4; footprint Connector_WUT:PinHeader_1x03_P2.54mm_Vertical -> Connector_Harwin_M20-999_WUT:M20-9990346; symbol Connector_WUT:Harwin_M20-9990346 -> connector_auto_wut:Harwin_M20-9990346; JLCPCB Order # (none) -> C5355646
- CN6: footprint Connector_JST:JST_SH_BM03B-SRSS-TB_1x03-1MP_P1.00mm_Vertical -> Connector_JST_WUT:BM03B-SRSS-TB; symbol Connector_WUT:Header_JST_BM03B-SRSS-TB(LF)(SN) -> connector_auto_wut:JST_BM03B-SRSS-TB(LF)(SN)
- CN7, CN8: footprint Connector_JST:JST_SH_BM04B-SRSS-TB_1x04-1MP_P1.00mm_Vertical -> Connector_JST_WUT:BM04B-SRSS-TB; symbol Connector_WUT:Header_JST_BM04B-SRSS-TB(LF)(SN) -> connector_auto_wut:JST_BM04B-SRSS-TB(LF)(SN)
- CN9: renamed from CN11; footprint Connector_JST:JST_SH_BM05B-SRSS-TB_1x05-1MP_P1.00mm_Vertical -> Connector_JST_WUT:BM05B-SRSS-TB; symbol Connector_WUT:Header_JST_BM05B-SRSS-TB(LF)(SN) -> connector_auto_wut:JST_BM05B-SRSS-TB(LF)(SN)
- FB2: renamed from FB3; footprint Inductor_SMD:L_0402_1005Metric -> Inductor_WUT:L_0402_1005Metric
- renumbered C47 to C15, C15 to C16, C16 to C17, C48 to C18, C45 to C19, C17 to C20, C18 to C21, C19 to C22, C20 to C23, C21 to C24, C22 to C25, C23 to C26, C24 to C27, C25 to C28, C26 to C29, C27 to C30, C28 to C31, C29 to C32, C46 to C33, C51 to C34, CN5 to CN2, CN2 to CN4, CN3 to CN5, D7 to D1, D8 to D10, D14 to D11, D15 to D12, D16 to D13, D17 to D14, D19 to D15, D9 to D2, D10 to D3, D1 to D4, D2 to D5, D3 to D6, D4 to D7, D5 to D8, D6 to D9, H3 to H10, H6 to H11, H7 to H12, H10 to H13, R14 to R10, R9 to R11, R10 to R12, R11 to R13, R12 to R14, R23 to R15, R24 to R16, R25 to R17, R26 to R18, R27 to R19, R28 to R20, R29 to R21, R30 to R22, R31 to R23, R15 to R24, R35 to R25, R36 to R26, R37 to R27, R38 to R28, R39 to R29, R40 to R30, R41 to R31, R42 to R32, R43 to R33, R44 to R34, R45 to R35, R46 to R36, R47 to R37, R48 to R38, R49 to R39, R50 to R40, R51 to R41, R52 to R42, R53 to R43, R54 to R44, R55 to R45, R56 to R46, R57 to R47, R32 to R48, R13 to R9, U3 to U2, U4 to U3, U2 to U4
Connections:
- net 0V: now also CN10.MP1 (MNT), CN10.MP2 (MNT), CN11.MP1 (MNT), CN11.MP2 (MNT), CN6.MP1 (MNT), CN6.MP2 (MNT), CN7.MP1 (MNT), CN7.MP2 (MNT), CN8.MP1 (MNT), CN8.MP2 (MNT), CN9.MP1 (MNT), CN9.MP2 (MNT)
Other:
- moved on the sheet: R26, R27, R28, R29, R30

Commit message: draft v1 release
Parts:
- removed FB2: 1k8, Inductor_WUT:L_0402_1005Metric, symbol aaa_ferrite_bead_auto_wut:Murata BLM15BD182SN1D
Connections:
- net VDDA is gone; now on net 3V3: C27.1, C29.1, C31.1, U4.20 (VREF+), U4.21 (VDDA)
- net at U4.44 (PE14): no longer names the net of U4.44 (PE14)
- no-connect marks 10 -> 27
Other:
- note added: "VDDA used for ADC,DAC,comp and op-amp. None of these are used so minimal filtering is fine."
