File: P0004-PCB-001.kicad_pcb (KiCad board)
At the start: 4 copper layers, 63.5 x 38.5 mm, 165 parts, among them CN1 Liansheng PH--00603, CN10 JST BM06B-SRSS-TB(LF)(SN), CN11 BM05B-SRSS-TB(LF)(SN), CN2 Samtec FTSH-107-01-L-DV-K, CN3 104031-0811, CN4 M20-9990346, CN5 Molex 105057-0001, CN6 BM03B-SRSS-TB(LF)(SN), CN7 BM04B-SRSS-TB(LF)(SN), CN8 BM04B-SRSS-TB(LF)(SN), CN9 JST BM06B-SRSS-TB(LF)(SN), SW1 Khon TSB06331-090D332DA-R0500, SW2 Khon TSB06331-090D332DA-R0500, SW3 Khon TSB06331-090D332DA-R0500, SW4 Khon TSB06331-090D332DA-R0500, U1 W5500, U2 STM32H743VIT6, U3 TMP102AIDRL, U4 Microchip 24AA256UIDT-I/ST, U5 TI LMR54410DBV, U6 TI LMR54410DBV, U7 TI TPS2553DBV

Commit message: just need last tidy up
Parts:
- removed R32, R33, R34: 1k0, Resistor_WUT:R_0402_1005Metric
- added C49: 100n, Capacitor_WUT:C_0402_1005Metric, F.Cu at (150.8, 110.2)
- added C50: 22u, Capacitor_SMD:C_0603_1608Metric, F.Cu at (152.0, 116.8)
- added D14: 5V, Diode_SMD:D_SOD-523, F.Cu at (200.8, 121.2)
- added D15: 5V, Diode_SMD:D_SOD-523, F.Cu at (172.8, 114.4)
- added D16: 5V, Diode_SMD:D_SOD-523, F.Cu at (170.2, 114.4)
- added D17: 5V, Diode_SMD:D_SOD-523, F.Cu at (154.2, 114.2)
- added R59: 47k, Resistor_WUT:R_0402_1005Metric, F.Cu at (150.8, 116.2)
- added R60: 10k, Resistor_WUT:R_0402_1005Metric, F.Cu at (149.2, 115.8)
- added U8: TI TPS2553DBVR-1, IC_WUT:SOT-23-6, F.Cu at (150.8, 113.0)
- C43, C44: value 15p -> 18p
- C45: value 10u -> 22u
- D1, D2, D3, D4, D5, D6, D7, D8, D9: value 3V3 -> 5V
- R21: value 47k -> 82k
- R4: value 1k0 -> 10k
- U7: value TI TPS2553DBV -> TI TPS2553DBVR-1
- moved R4 11.3 mm to (181.5, 102.5)
- moved R6 1.00 mm to (179.2, 113.8)
- moved R7 1.00 mm to (180.2, 113.8)
- moved R53 0.71 mm to (159.8, 111.2), turned to 180 degrees
- moved C18 0.25 mm to (161.5, 104.2)
- moved C24 0.25 mm to (162.0, 107.8)
- moved C26 0.25 mm to (161.0, 109.8)
- moved C28 0.25 mm to (162.0, 109.8)
- moved C29 0.25 mm to (161.5, 106.2)
- moved C33 0.25 mm to (198.0, 118.0)
- moved C37 0.25 mm to (199.0, 118.0)
- moved C40 0.25 mm to (199.0, 116.2)
- moved C7 0.25 mm to (182.8, 113.2)
- moved C9 0.25 mm to (182.8, 114.2)
- moved FB3 0.25 mm to (161.0, 107.8)
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Connections:
- net Net-(U1-TXN) renamed /Ethernet/TX_N
- net Net-(U1-TXP) renamed /Ethernet/TX_P
- C46 pad 1: /Microcontroller/DFU_EN -> /DFU_EN
- CN1 pad 1: unconnected-(CN1-Pin_1-Pad1) -> /VIN
- CN1 pad 10: unconnected-(CN1-Pad10) -> 0V
- CN1 pad 11: unconnected-(CN1-Pad11) -> /ETH_TX_N
- CN1 pad 12: unconnected-(CN1-Pad12) -> 0V
- CN1 pad 13: unconnected-(CN1-Pad13) -> /~{ETH_LINK_OD}
- CN1 pad 14: unconnected-(CN1-Pad14) -> 0V
- CN1 pad 15: unconnected-(CN1-Pad15) -> /~{ETH_ACT_OD}
- CN1 pad 16: unconnected-(CN1-Pad16) -> 0V
- CN1 pad 17: unconnected-(CN1-Pad17) -> /INT_SDA
- CN1 pad 18: unconnected-(CN1-Pad18) -> 0V
- CN1 pad 19: unconnected-(CN1-Pad19) -> /INT_SCL
- CN1 pad 2: unconnected-(CN1-Pin_1-Pad2) -> 0V
- CN1 pad 20: unconnected-(CN1-Pad20) -> 0V
- CN1 pad 21: unconnected-(CN1-Pad21) -> /USB_P
- CN1 pad 22: unconnected-(CN1-Pad22) -> 0V
- CN1 pad 23: unconnected-(CN1-Pad23) -> /USB_N
- CN1 pad 24: unconnected-(CN1-Pad24) -> 0V
- CN1 pad 25: unconnected-(CN1-Pad25) -> /DFU_EN
- CN1 pad 26: unconnected-(CN1-Pad26) -> 0V
- CN1 pad 27: unconnected-(CN1-Pad27) -> /~{INT_ALERT}
- CN1 pad 28: unconnected-(CN1-Pad28) -> 0V
- CN1 pad 29: unconnected-(CN1-Pad29) -> 3V3_EXPANSION
- CN1 pad 3: unconnected-(CN1-Pad3) -> 0V
- CN1 pad 30: unconnected-(CN1-Pad30) -> 0V
- CN1 pad 4: unconnected-(CN1-Pad4) -> 0V
- CN1 pad 5: unconnected-(CN1-Pad5) -> /ETH_RX_P
- CN1 pad 6: unconnected-(CN1-Pad6) -> 0V
- CN1 pad 7: unconnected-(CN1-Pad7) -> /ETH_RX_N
- CN1 pad 8: unconnected-(CN1-Pad8) -> 0V
- CN1 pad 9: unconnected-(CN1-Pad9) -> /ETH_TX_P
- F2 pad 1: /Power Supplies/VIN -> /VIN
- R35 pad 1: /Microcontroller/DFU_EN -> /DFU_EN
- R4 pad 2: Net-(R33-Pad1) -> /Ethernet/~{ETH_PHY_RST}
- R5 pad 1: /Ethernet/ETH_RX_N -> /ETH_RX_P
- R6 pad 2: /Ethernet/ETH_TX_P -> /ETH_TX_N
- R7 pad 2: /Ethernet/ETH_TX_N -> /ETH_TX_P
- R8 pad 1: /Ethernet/ETH_RX_P -> /ETH_RX_N
- SW1 pad 2: unconnected-(SW1-Pad2) -> 0V
- SW1 pad 3: unconnected-(SW1-Pad3) -> /Microcontroller/~{SW1}
- SW2 pad 2: unconnected-(SW2-Pad2) -> /Microcontroller/~{SW2}
- SW2 pad 3: unconnected-(SW2-Pad3) -> 0V
- SW2 pad 4: unconnected-(SW2-Pad4) -> 0V
- SW3 pad 1: unconnected-(SW3-Pad1) -> /Microcontroller/~{SW3}
- SW3 pad 3: unconnected-(SW3-Pad3) -> 0V
- SW3 pad 4: unconnected-(SW3-Pad4) -> 0V
- SW4 pad 1: unconnected-(SW4-Pad1) -> /Microcontroller/~{SW4}
- SW4 pad 3: unconnected-(SW4-Pad3) -> 0V
- SW4 pad 4: unconnected-(SW4-Pad4) -> 0V
- U1 pad 25: /Ethernet/~{ETH_LINK_OD} -> /~{ETH_LINK_OD}
- U1 pad 27: /Ethernet/~{ETH_ACT_OD} -> /~{ETH_ACT_OD}
- U1 pad 5: /Ethernet/ETH_RX_P -> /ETH_RX_N
- U1 pad 6: /Ethernet/ETH_RX_N -> /ETH_RX_P
- U2 pad 38: unconnected-(U2-PE8-Pad38) -> /Microcontroller/~{3V3_EXPANSION_FAULT}
- U2 pad 39: unconnected-(U2-PE9-Pad39) -> /Microcontroller/~{SW3}
- U2 pad 40: unconnected-(U2-PE10-Pad40) -> /Microcontroller/~{SW1}
- U2 pad 42: unconnected-(U2-PE12-Pad42) -> /Microcontroller/~{SW2}
- U2 pad 43: unconnected-(U2-PE13-Pad43) -> /Microcontroller/~{SW4}
- U2 pad 53: /Microcontroller/USB_DEVICE_D_N -> /USB_N
- U2 pad 54: /Microcontroller/USB_DEVICE_D_P -> /USB_P
- U2 pad 58: /Microcontroller/~{INT_ALERT} -> /~{INT_ALERT}
- U2 pad 94: /Microcontroller/DFU_EN -> /DFU_EN
- U3 pad 3: /Microcontroller/~{INT_ALERT} -> /~{INT_ALERT}
Routing:
- net /~{INT_ALERT}: track 0.00 -> 68.3 mm, vias 0 -> 3
- net /Microcontroller/~{SW1}: track 0.00 -> 39.7 mm, vias 0 -> 2
- net /DFU_EN: track 0.00 -> 31.7 mm, vias 0 -> 2
- net /Microcontroller/~{3V3_EXPANSION_FAULT}: track 0.00 -> 30.6 mm, vias 0 -> 2
- net /Microcontroller/~{INT_ALERT}: track 28.1 -> 0.00 mm, vias 2 -> 0
- net /USB_P: track 0.00 -> 26.0 mm, vias 0 -> 2
- net /Microcontroller/~{SW4}: track 0.00 -> 25.9 mm, vias 0 -> 2
- net /USB_N: track 0.00 -> 25.4 mm, vias 0 -> 2
- net /~{ETH_ACT_OD}: track 0.00 -> 22.6 mm, vias 0 -> 2
- net /Microcontroller/INT_SCL: track 8.18 -> 30.3 mm, vias 1 -> 2
- net /~{ETH_LINK_OD}: track 0.00 -> 21.5 mm, vias 0 -> 2
- net /Microcontroller/INT_SDA: track 6.92 -> 26.6 mm, vias 1 -> 2
- net 0V: track 95.1 -> 80.9 mm, vias 146 -> 186
- net /Microcontroller/~{SW2}: track 0.00 -> 11.2 mm, vias 0 -> 1
- net unconnected-(U2-PE7-Pad37): track 6.86 -> 0.00 mm, vias 1 -> 0
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- added copper zone on B.Cu, net 0V
- added copper zone on In3.Cu, net 0V
- added copper zone on In4.Cu, net 0V
- added copper zone on In3.Cu, net 3V3
- added copper zone on In3.Cu, net 5V_VBUS
- removed copper zone on B.Cu, net 3V3
Other:
- copper layers 4 -> 6
- board text removed: "FUET-5020"

Commit message: component tidy up
Parts:
- removed the D11 at (194.8, 113.5)
- added C34: 22u, Capacitor_WUT:C_0603_1608Metric, F.Cu at (152.5, 122.2)
- added D15: B2020WS, Diode_WUT:D_SOD-323, F.Cu at (152.5, 119.0)
- added D16: 15V, Diode_WUT:D_SOD-323, F.Cu at (194.9, 113.5)
- added Q1: BC847C,215, IC_WUT:SOT-23, F.Cu at (149.8, 116.0)
- added R48: 1k0, Resistor_WUT:R_0402_1005Metric, F.Cu at (147.2, 116.0)
- C17: renamed from C16; footprint Capacitor_SMD:C_0603_1608Metric -> Capacitor_WUT:C_0603_1608Metric
- C19: renamed from C45; footprint Capacitor_SMD:C_0603_1608Metric -> Capacitor_WUT:C_0603_1608Metric
- C40: renamed from C35; footprint Capacitor_SMD:C_0603_1608Metric -> Capacitor_WUT:C_0603_1608Metric
- C41: renamed from C36; footprint Capacitor_SMD:C_0603_1608Metric -> Capacitor_WUT:C_0603_1608Metric
- C44: renamed from C39; footprint Capacitor_SMD:C_0603_1608Metric -> Capacitor_WUT:C_0603_1608Metric
- C45: renamed from C40; footprint Capacitor_SMD:C_0603_1608Metric -> Capacitor_WUT:C_0603_1608Metric
- C46: renamed from C41; footprint Capacitor_SMD:C_0603_1608Metric -> Capacitor_WUT:C_0603_1608Metric
- C47: renamed from C42; footprint Capacitor_SMD:C_0603_1608Metric -> Capacitor_WUT:C_0603_1608Metric
- C51: renamed from C50; footprint Capacitor_SMD:C_0603_1608Metric -> Capacitor_WUT:C_0603_1608Metric
- D1: renamed from D7; footprint Diode_SMD:D_SOD-523 -> Diode_WUT:D_SOD-523
- D10: renamed from D8; footprint Diode_SMD:D_SOD-523 -> Diode_WUT:D_SOD-523
- D11: renamed from D14; footprint Diode_SMD:D_SOD-523 -> Diode_WUT:D_SOD-523
- D12: renamed from D15; footprint Diode_SMD:D_SOD-523 -> Diode_WUT:D_SOD-523
- D13: renamed from D16; footprint Diode_SMD:D_SOD-523 -> Diode_WUT:D_SOD-523
- D14: renamed from D17; footprint Diode_SMD:D_SOD-523 -> Diode_WUT:D_SOD-523
- D17: renamed from D12; footprint Diode_SMD:D_SOD-523 -> Diode_WUT:D_SOD-523
- D18: renamed from D13; footprint Diode_SMD:D_SOD-523 -> Diode_WUT:D_SOD-523
- D2: renamed from D9; footprint Diode_SMD:D_SOD-523 -> Diode_WUT:D_SOD-523
- D3: renamed from D10; footprint Package_TO_SOT_SMD:SOT-666 -> IC_WUT:SOT-666
- D4: renamed from D1; footprint Diode_SMD:D_SOD-523 -> Diode_WUT:D_SOD-523
- D5: renamed from D2; footprint Diode_SMD:D_SOD-523 -> Diode_WUT:D_SOD-523
- D6: renamed from D3; footprint Diode_SMD:D_SOD-523 -> Diode_WUT:D_SOD-523
- D7: renamed from D4; footprint Diode_SMD:D_SOD-523 -> Diode_WUT:D_SOD-523
- D8: renamed from D5; footprint Diode_SMD:D_SOD-523 -> Diode_WUT:D_SOD-523
- D9: renamed from D6; footprint Diode_SMD:D_SOD-523 -> Diode_WUT:D_SOD-523
- F1, F2, F3, F4: footprint Fuse:Fuse_0603_1608Metric -> Fuse_WUT:Fuse_0603_1608Metric
- LS1: value HNDZ MLT8530 -> Fusheng FUET-5020; footprint Audio_WUT:HNDZ_MLT8530 -> Audio_WUT:Fusheng_FUET-5020
- moved LS1 12.8 mm to (148.5, 120.8)
- moved R56 5.22 mm to (149.2, 111.2), turned to 90 degrees
- moved C51 4.72 mm to (156.0, 114.2), turned to 0 degrees
- moved R57 2.50 mm to (149.2, 113.2), turned to 90 degrees
- moved D14 2.47 mm to (152.5, 116.0), turned to 90 degrees
- moved R43 1.77 mm to (161.5, 111.0)
- moved C50 1.68 mm to (152.2, 109.5)
- moved U8 1.07 mm to (151.5, 112.2)
- moved C21 0.25 mm to (161.5, 104.0)
- moved C27 0.25 mm to (162.0, 107.5)
- moved C29 0.25 mm to (161.0, 109.5)
- moved C31 0.25 mm to (162.0, 109.5)
- moved C32 0.25 mm to (161.5, 106.0)
- moved FB2 0.25 mm to (161.0, 107.5)
- moved R24 0.25 mm to (161.5, 105.0)
- renumbered C47 to C15, C15 to C16, C48 to C18, C17 to C20, C18 to C21, C19 to C22, C20 to C23, C21 to C24, C22 to C25, C23 to C26, C24 to C27, C25 to C28, C26 to C29, C27 to C30, C28 to C31, C29 to C32, C46 to C33, C30 to C35, C31 to C36, C32 to C37, C33 to C38, C34 to C39, C37 to C42, C38 to C43, C43 to C48, C44 to C49, C49 to C50, CN9 to CN10, CN10 to CN11, CN5 to CN2, CN4 to CN3, CN2 to CN4, CN3 to CN5, CN11 to CN9, FB3 to FB2, H3 to H10, H6 to H11, H7 to H12, H10 to H13, H4 to H3, H5 to H4, H8 to H5, H9 to H6, H11 to H7, H12 to H8, H13 to H9, R14 to R10, R9 to R11, R10 to R12, R11 to R13, R12 to R14, R23 to R15, R24 to R16, R25 to R17, R26 to R18, R27 to R19, R28 to R20, R29 to R21, R30 to R22, R31 to R23, R15 to R24, R35 to R25, R36 to R26, R37 to R27, R38 to R28, R39 to R29, R40 to R30, R41 to R31, R42 to R32, R43 to R33, R44 to R34, R45 to R35, R46 to R36, R47 to R37, R48 to R38, R49 to R39, R50 to R40, R51 to R41, R52 to R42, R53 to R43, R54 to R44, R55 to R45, R56 to R46, R57 to R47, R16 to R49, R17 to R50, R18 to R51, R19 to R52, R20 to R53, R21 to R54, R22 to R55, R59 to R56, R60 to R57, R8 to R6, R6 to R7, R7 to R8, R13 to R9, U3 to U2, U4 to U3, U2 to U4
Connections:
- LS1 pad 1: unconnected-(LS1-+-Pad1) -> 3V3
- LS1 pad 2: unconnected-(LS1---Pad2) -> Net-(D15-A)
- R44 pad 1: /Microcontroller/PB0 -> /Microcontroller/PC5
- U4 pad 33: unconnected-(U2-PC5-Pad33) -> /Microcontroller/PC5
- U4 pad 34: /Microcontroller/PB0 -> /Microcontroller/SPEAKER
Routing:
- net /Microcontroller/SPEAKER: track 0.00 -> 34.3 mm, vias 0 -> 2
- net /Microcontroller/PC5: track 0.00 -> 14.2 mm, vias 0 -> 2
- net /Microcontroller/PB0: track 13.7 -> 0.00 mm, vias 2 -> 0
- net 0V: track 80.9 -> 74.9 mm, vias 186 -> 183
- net Net-(D15-A): track 0.00 -> 5.90 mm
- net 3V3_EXPANSION: track 5.11 -> 0.00 mm
- net 3V3: track 43.3 -> 40.2 mm, vias 30 -> 32
- net /Microcontroller/~{3V3_EXPANSION_FAULT}: track 30.6 -> 33.3 mm
- net /Microcontroller/SPI6_MOSI: track 45.4 -> 42.9 mm
- net /Microcontroller/~{SW4}: track 25.9 -> 27.9 mm
- net Net-(U8-ILIM): track 1.60 -> 3.47 mm
- net /Microcontroller/PA3: track 3.42 -> 1.57 mm
- net Net-(Q1-B): track 0.00 -> 1.74 mm
- net Net-(CN11-Pin_2-Pad2): track 2.82 -> 4.47 mm
- net /Microcontroller/VDDA: track 6.41 -> 7.72 mm
- added copper zone on F.Cu, net 3V3_EXPANSION
- removed copper zone on In3.Cu, net 0V

Commit message: added tidied up library symbols
Parts:
- CN10, CN11: value JST BM06B-SRSS-TB(LF)(SN) -> BM06B-SRSS-TB(LF)(SN); footprint Connector_JST:JST_SH_BM06B-SRSS-TB_1x06-1MP_P1.00mm_Vertical -> Connector_JST_WUT:BM06B-SRSS-TB
- CN3: footprint Connector_WUT:PinHeader_1x03_P2.54mm_Vertical -> Connector_Harwin_M20-999_WUT:M20-9990346
- CN6: footprint Connector_JST:JST_SH_BM03B-SRSS-TB_1x03-1MP_P1.00mm_Vertical -> Connector_JST_WUT:BM03B-SRSS-TB
- CN7, CN8: footprint Connector_JST:JST_SH_BM04B-SRSS-TB_1x04-1MP_P1.00mm_Vertical -> Connector_JST_WUT:BM04B-SRSS-TB
- CN9: footprint Connector_JST:JST_SH_BM05B-SRSS-TB_1x05-1MP_P1.00mm_Vertical -> Connector_JST_WUT:BM05B-SRSS-TB
- FB1: footprint Inductor_SMD:L_0603_1608Metric -> Inductor_WUT:L_0603_1608Metric
- FB2: footprint Inductor_SMD:L_0402_1005Metric -> Inductor_WUT:L_0402_1005Metric
- moved CN3 2.54 mm to (169.8, 89.8), turned to -90 degrees
- moved CN10 0.50 mm to (155.5, 98.2)
- moved CN11 0.50 mm to (155.5, 108.2)
- moved CN6 0.50 mm to (149.0, 106.8)
- moved CN7 0.50 mm to (158.5, 89.5)
- moved CN8 0.50 mm to (151.0, 89.5)
- moved CN9 0.50 mm to (149.0, 98.2)
Routing:
- net /~{INT_ALERT}: track 68.3 -> 59.1 mm
- net /USB_P: track 26.0 -> 31.6 mm
- net /USB_N: track 25.4 -> 31.0 mm
- net 0V: track 74.9 -> 75.9 mm, vias 183 -> 187
