File: P0004-PCB-001.kicad_pcb (KiCad board)
At the start: 6 copper layers, 63.5 x 38.5 mm, 175 parts, among them CN1 Liansheng PH--00603, CN10 BM06B-SRSS-TB(LF)(SN), CN11 BM06B-SRSS-TB(LF)(SN), CN2 Molex 105057-0001, CN3 M20-9990346, CN4 Samtec FTSH-107-01-L-DV-K, CN5 104031-0811, CN6 BM03B-SRSS-TB(LF)(SN), CN7 BM04B-SRSS-TB(LF)(SN), CN8 BM04B-SRSS-TB(LF)(SN), CN9 BM05B-SRSS-TB(LF)(SN), Q1 BC847C,215, SW1 Khon TSB06331-090D332DA-R0500, SW2 Khon TSB06331-090D332DA-R0500, SW3 Khon TSB06331-090D332DA-R0500, SW4 Khon TSB06331-090D332DA-R0500, U1 W5500, U2 TMP102AIDRL, U3 Microchip 24AA256UIDT-I/ST, U4 STM32H743VIT6, U5 TI LMR54410DBV, U6 TI LMR54410DBV, U7 TI TPS2553DBVR-1, U8 TI TPS2553DBVR-1

Commit message: draft v1 release
Parts:
- removed FB2: 1k8, Inductor_WUT:L_0402_1005Metric
- moved H9 2.00 mm to (189.5, 98.8)
- moved D6 0.25 mm to (181.0, 94.8)
- moved D7 0.25 mm to (183.5, 94.8)
- moved D16 0.10 mm to (194.9, 113.6)
- moved L2 0.10 mm to (198.8, 110.8)
Connections:
- C27 pad 1: /Microcontroller/VDDA -> 3V3
- C29 pad 1: /Microcontroller/VDDA -> 3V3
- C31 pad 1: /Microcontroller/VDDA -> 3V3
- U2 pad 1: /Microcontroller/INT_SCL -> /INT_SCL
- U2 pad 6: /Microcontroller/INT_SDA -> /INT_SDA
- U3 pad 5: /Microcontroller/INT_SDA -> /INT_SDA
- U3 pad 6: /Microcontroller/INT_SCL -> /INT_SCL
- U4 pad 20: /Microcontroller/VDDA -> 3V3
- U4 pad 21: /Microcontroller/VDDA -> 3V3
- U4 pad 44: /Microcontroller/<NO NET> -> unconnected-(U4-PE14-Pad44)
- U4 pad 59: /Microcontroller/INT_SCL -> /INT_SCL
- U4 pad 60: /Microcontroller/INT_SDA -> /INT_SDA
Routing:
- net /INT_SCL: track 0.00 -> 55.8 mm, vias 0 -> 3
- net /INT_SDA: track 0.00 -> 51.1 mm, vias 0 -> 3
- net /Microcontroller/INT_SCL: track 30.3 -> 0.00 mm, vias 2 -> 0
- net /Microcontroller/INT_SDA: track 26.6 -> 0.00 mm, vias 2 -> 0
- net /Microcontroller/VDDA: track 7.71 -> 0.00 mm
- net 3V3: track 40.4 -> 47.5 mm, vias 32 -> 33
- net /VIN: track 2.52 -> 6.30 mm
- net 0V: track 75.9 -> 72.4 mm
- net /USB_P: track 31.6 -> 29.6 mm
- net /Ethernet/PHY_VDDA: track 12.7 -> 14.8 mm
- net /USB_N: track 31.0 -> 29.1 mm
- net /Microcontroller/~{3V3_EXPANSION_FAULT}: track 33.3 -> 31.6 mm
- net /Microcontroller/~{I2C2_ALERT}: track 43.3 -> 42.3 mm
- net /Microcontroller/SPEAKER: track 34.3 -> 33.4 mm
- net 5V_VBUS: vias 12 -> 11
- added copper zone on In3.Cu, net 0V
- added copper zone on In4.Cu, net 3V3
- added copper zone on In4.Cu, net 5V_VBUS
- removed copper zone on In4.Cu, net 0V
- removed copper zone on In3.Cu, net 3V3
- removed copper zone on B.Cu, net 5V_VBUS
- removed copper zone on In3.Cu, net 5V_VBUS
Other:
- board text added: "Use JLC0616H-3313 stackup"
